File: TPMS Board design.kicad_sch (KiCad schematic)
At the start: 22 parts, among them J1 CAN_IN, J2 CAN_OUT, J3 CAN_DB9, U1 ADM3055E, U2 ESP32-C3, U3 CDSOT23-T24CAN, Y2 Crystal

Commit message: Update
Connections:
- net +3V3 is gone; now on net +3.3V: C3.1, C4.1, U1.4 (V_IO), U2.11 (VDD3P3_RTC), U2.17 (VDD3P3_CPU), U2.18 (VDD_SPI), U2.2 (VDD3P3), U2.3 (VDD3P3__1), U2.31 (VDDA), U2.32 (VDDA__1)
Changed lines of the file:
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@@
 			)
 		)
-		(property "Value" "+3V3"
+		(property "Value" "+3.3V"
 			(at 99.441 121.3358 0)
 			(effects
@@
 			)
 		)
-		(property "Value" "+3V3"
+		(property "Value" "+3.3V"
 			(at 116.84 31.7499 90)
 			(effects

Commit message: IC
Other:
- moved on the sheet: C10, C11
Changed lines of the file:
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@@
 	(wire
 		(pts
-			(xy 19.05 48.26) (xy 15.24 48.26)
+			(xy 17.78 48.26) (xy 15.24 48.26)
 		)
 		(stroke
@@
 	(wire
 		(pts
-			(xy 15.24 55.88) (xy 19.05 55.88)
+			(xy 15.24 55.88) (xy 21.59 55.88)
 		)
 		(stroke
@@
 	(wire
 		(pts
-			(xy 26.67 48.26) (xy 31.75 48.26)
+			(xy 25.4 48.26) (xy 31.75 48.26)
 		)
 		(stroke
@@
 	(wire
 		(pts
-			(xy 26.67 55.88) (xy 31.75 55.88)
+			(xy 29.21 55.88) (xy 31.75 55.88)
 		)
 		(stroke
@@
 	(symbol
 		(lib_id "Device:C")
-		(at 22.86 48.26 90)
+		(at 21.59 48.26 90)
 		(unit 1)
 		(exclude_from_sim no)
@@
 		(dnp no)
 		(property "Reference" "C10"
-			(at 22.86 42.164 90)
+			(at 21.59 42.164 90)
 			(effects
 				(font
@@
 		)
 		(property "Value" "18Pf"
-			(at 22.86 44.704 90)
+			(at 21.59 44.704 90)
 			(effects
 				(font
@@
 		)
 		(property "Footprint" "Capacitor_SMD:C_0805_2012Metric"
-			(at 26.67 47.2948 0)
+			(at 25.4 47.2948 0)
 			(effects
 				(font
@@
 		)
 		(property "Datasheet" "~"
-			(at 22.86 48.26 0)
+			(at 21.59 48.26 0)
 			(effects
 				(font
@@
 		)
 		(property "Description" "Unpolarized capacitor"
-			(at 22.86 48.26 0)
+			(at 21.59 48.26 0)
 			(effects
 				(font
@@
 	(symbol
 		(lib_id "Device:C")
-		(at 22.86 55.88 90)
+		(at 25.4 55.88 90)
 		(unit 1)
 		(exclude_from_sim no)
@@
 		(dnp no)
 		(property "Reference" "C11"
-			(at 22.86 59.436 90)
+			(at 25.4 59.436 90)
 			(effects
 				(font
@@
 		)
 		(property "Value" "18pf"
-			(at 23.114 62.23 90)
+			(at 25.654 62.23 90)
 			(effects
 				(font
@@
 		)
 		(property "Footprint" "Capacitor_SMD:C_0805_2012Metric"
-			(at 26.67 54.9148 0)
+			(at 29.21 54.9148 0)
 			(effects
 				(font
@@
 		)
 		(property "Datasheet" "~"
-			(at 22.86 55.88 0)
+			(at 25.4 55.88 0)
 			(effects
 				(font
@@
 		)
 		(property "Description" "Unpolarized capacitor"
-			(at 22.86 55.88 0)
+			(at 25.4 55.88 0)
 			(effects
 				(font
